File: PCB/flight_controller/flight_controller.kicad_sch (KiCad schematic)
At the start: 5 parts, among them J3 Conn_01x04_Socket_JST_ELRS, J4 Conn_01x10_Socket_JST_ESC, U1 module_mpu6050, U2 ESP32-DevKitC

Commit message: wip
Parts:
- added H1, H2, H3, H4: MountingHole, MountingHole:MountingHole_2.2mm_M2, symbol Mechanical:MountingHole
- J3: footprint (none) -> Connector_JST:JST_SH_SM04B-SRSS-TB_1x04-1MP_P1.00mm_Horizontal
- J4: footprint (none) -> Connector_JST:JST_SH_SM10B-SRSS-TB_1x10-1MP_P1.00mm_Horizontal
- U2: footprint PCM_Espressif:ESP32-DevKitC -> ESP32:ESP32 DevKitC Socket
- renumbered MP to MP1
Connections:
- net GND: now reaches J3.1 (Pin_1)
- net GND: now also J4.1 (Pin_1), J4.2 (Pin_2), MP1.2 (VIN-), MP1.4 (VOUT-), U1.2 (GND), U2.14 (GND), U2.32 (GND), U2.38 (GND)
- net VCC: now reaches J3.2 (Pin_2)
- net VCC: now also U1.1 (VCC), U2.1 (3V3)
- net TX: now reaches J3.3 (Pin_3)
- net TX: now also U2.27 (GPIO16)
- net RX: now reaches J3.4 (Pin_4)
- net RX: now also U2.28 (GPIO17)
- net ESC1: now reaches U2.12 (MTMS/GPIO14/ADC2_CH6)
- net ESC1: now also J4.8 (Pin_8)
- net ESC2: now reaches U2.13 (MTDI/GPIO12/ADC2_CH5)
- net ESC2: now also J4.7 (Pin_7)
- net ESC3: now reaches U2.15 (MTCK/GPIO13/ADC2_CH4)
- net ESC3: now also J4.6 (Pin_6)
- net at U2.19 (5V): now also MP1.3 (VOUT+)
- net ESC4: now reaches U2.23 (MTDO/GPIO15/ADC2_CH3)
- net ESC4: now also J4.5 (Pin_5)
- net at U2.33 (GPIO21): now also U1.4 (SDA)
- net at U2.36 (GPIO22): now also U1.3 (SCL)
- net 10V: now reaches J4.4 (Pin_4)
- net 10V: now also MP1.1 (VIN+)
- no-connect marks 0 -> 32
Other:
- moved on the sheet: J3, J4, MP1, U1, U2
